Commit message: change 20.04 hp VM

File: arduinobot_description/urdf/arduinobot.urdf.xacro (robot description, xacro)
@@ -5,8 +5,29 @@
     <xacro:property name="effort" value="30" />
     <xacro:property name="velocity" value="10" />
+    <xacro:macro name="default_inertial" params="mass">
+        <inertial>
+            <mass value="${mass}"/>
+            <inertia ixx="1.0" ixy="0.0" ixz="0.0" iyy="1.0" iyz="0.0" izz="1.0"/>
+        </inertial>
+    </xacro:macro>
+    <xacro:macro name="default_transmission" params="number">
+        <transmission name = "transmission_${number}" >
+            <type>
+                transmission_interface/SimpleTransmission
+            </type>
+            <joint name="joint_${number}">
+                <hardwareInterface>hardware_interface/PositionJointInterface</hardwareInterface>
+            </joint>
+            <actuator name="motor_${number}">
+                <hardwareInterface>hardware_interface/PositionJointInterface</hardwareInterface>
+                <mechanicalReduction>1</mechanicalReduction>
+            </actuator>
+        </transmission>
+    </xacro:macro>
     <!-- Links -->
     <link name="world"/>
     <!-- Link 1 -->
     <link name="base_link">
+        <xacro:default_inertial mass = "1.0"/>
         <visual>
             <origin rpy="0 0 0" xyz="-0.5 -0.5 0"/>
@@ -18,4 +39,5 @@
     <!-- Link 2 -->
     <link name="base_plate">
+        <xacro:default_inertial mass = "0.1"/>
         <visual>
             <origin rpy="0 0 0" xyz="-0.39 -0.39 -0.56"/>
@@ -24,7 +46,14 @@
             </geometry>
         </visual>
+        <collision>
+            <origin rpy="0 0 0" xyz="-0.39 -0.39 -0.56"/>
+            <geometry>
+                <mesh filename="package://arduinobot_description/mesh/base_plate.STL" scale="0.01 0.01 0.01"/>
+            </geometry>
+        </collision>
     </link>
     <!-- Link 3 -->
     <link name="forward_drive_arm">
+        <xacro:default_inertial mass = "0.1"/>
         <visual>
             <origin rpy="0 -${PI/2} ${PI/2}" xyz="0.19 0.06 -0.08"/>
@@ -33,7 +62,14 @@
             </geometry>
         </visual>
+        <collision>
+            <origin rpy="0 -${PI/2} ${PI/2}" xyz="0.19 0.06 -0.08"/>
+            <geometry>
+                <mesh filename="package://arduinobot_description/mesh/forward_drive_arm.STL" scale="0.01 0.01 0.01"/>
+            </geometry>
+        </collision>
     </link>
     <!-- Link 4 -->
     <link name="horizontal_arm">
+        <xacro:default_inertial mass = "0.1"/>
         <visual>
             <origin rpy="${PI/2} 0 ${PI/2}" xyz="-0.03 -0.4 -0.06"/>
@@ -42,7 +78,14 @@
             </geometry>
         </visual>
+        <collision>
+            <origin rpy="${PI/2} 0 ${PI/2}" xyz="-0.03 -0.4 -0.06"/>
+            <geometry>
+                <mesh filename="package://arduinobot_description/mesh/horizontal_arm.STL" scale="0.01 0.01 0.01"/>
+            </geometry>
+        </collision>
     </link>
     <!-- Link 5 -->
     <link name="claw_support">
+        <xacro:default_inertial mass = "0.05"/>
         <visual>
             <origin rpy="0 0 ${PI/2}" xyz="0 -0.05 -0.15"/>
@@ -51,7 +94,14 @@
             </geometry>
         </visual>
+        <collision>
+            <origin rpy="0 0 ${PI/2}" xyz="0 -0.05 -0.15"/>
+            <geometry>
+                <mesh filename="package://arduinobot_description/mesh/claw_support.STL" scale="0.01 0.01 0.01"/>
+            </geometry>
+        </collision>
     </link>
     <!-- Link 6 -->
     <link name="gripper_right">
+        <xacro:default_inertial mass = "0.01"/>
         <visual>
             <origin rpy="0 0 -${PI/2}" xyz="-0.1 0.5 -0.1"/>
@@ -60,7 +110,14 @@
             </geometry>
         </visual>
+        <collision>
+            <origin rpy="0 0 -${PI/2}" xyz="-0.1 0.5 -0.1"/>
+            <geometry>
+                <mesh filename="package://arduinobot_description/mesh/right_finger.STL" scale="0.01 0.01 0.01"/>
+            </geometry>
+        </collision>
     </link>
     <!-- Link 7 -->
     <link name="gripper_left">
+        <xacro:default_inertial mass = "0.01"/>
         <visual>
             <origin rpy="0 0 -${PI/2}" xyz="-0.04 0.5 -0.1"/>
@@ -69,4 +126,10 @@
             </geometry>
         </visual>
+        <collision>
+            <origin rpy="0 0 -${PI/2}" xyz="-0.04 0.5 -0.1"/>
+            <geometry>
+                <mesh filename="package://arduinobot_description/mesh/left_finger.STL" scale="0.01 0.01 0.01"/>
+            </geometry>
+        </collision>
     </link>
     <!-- Link 8 -->
@@ -132,3 +195,27 @@
         <origin rpy="0.0 0.0 0.0" xyz="0 0 0"/>
     </joint>
+    <xacro:default_transmission number="1"/>
+    <xacro:default_transmission number="2"/>
+    <xacro:default_transmission number="3"/>
+    <xacro:default_transmission number="4"/>
+    <gazebo>
+        <plugin name="gazebo_ros_control" filename="libgazebo_ros_control.so">
+            <robotNamespace>/arduinobot</robotNamespace>
+            <robotSimType>gazebo_ros_control/DefaultRobotHWSim</robotSimType>
+            <legacyModeNS>true</legacyModeNS>
+        </plugin>
+        <!-- <plugin name="gazebo_ros_control" filename="libgazebo_ros_control.so">
+            <robotNamespace>/arduinobot</robotNamespace>
+            <robotSimType>gazebo_ros_control/DefaultRobotHWSim</robotSimType>
+            <legacyModeNS>true</legacyModeNS>
+        </plugin> -->
+        <plugin name="joint_5_mimic_joint_4" filename="libroboticsgroup_gazebo_mimic_joint_plugin.so">
+            <joint>joint_4</joint>
+            <mimicJoint>joint_5</mimicJoint>
+            <multiplier>-1.0</multiplier>
+            <offset>0</offset>
+            <maxEffort>${effort}</maxEffort>]
+            <robotNamespace>/arduinobot</robotNamespace>
+        </plugin>
+    </gazebo>
 </robot>
